Commit message: shop1 model

File: models/shopping_cart/automatic_cart.urdf.xacro (robot description, xacro)
@@ -1,8 +1,9 @@
 <?xml version="1.0"?>
 <robot name="automatic_cart" xmlns:xacro="http://ros.org/wiki/xacro">
-  <!-- Robot Body -->
+  <!-- Colors -->
   <material name="black">
     <color rgba="0 0 0 1"/>
   </material>
+  <!-- Robot params -->
   <xacro:property name="baseshift" value="0.2" />
   <xacro:property name="wheellen" value="0.025" />
@@ -17,4 +18,8 @@
   <xacro:property name="zwheel2" value="-0.15" />
   <xacro:property name="pi" value="3.1415" />
+  <!-- Sensor params -->
+  <xacro:arg name="laser_visual" default="false"/>
+  <xacro:arg name="imu_visual"   default="false"/>
+  <!-- Physic params -->
   <xacro:macro name="default_inertial" params="mass">
     <inertial>
@@ -29,4 +34,6 @@
     </inertial>
   </xacro:macro>
+  <!-- Robot Design -->
+  <link name="base_footprint"/>
   <link name="base_link">
     <visual>
@@ -42,6 +49,11 @@
       <origin rpy="0 0 ${pi}" xyz="0.0 0.0 ${baseshift}"/>
     </collision>
-    <xacro:default_inertial mass="30"/>
-  </link>
+    <xacro:default_inertial mass="10"/>
+  </link>
+  <joint name="base_joint" type="fixed">
+    <parent link="base_footprint"/>
+    <child link="base_link"/>
+    <origin xyz="0.0 0.0 0.0"/>
+  </joint>
   <link name="basket">
     <visual>
@@ -57,5 +69,5 @@
       <origin rpy="0 0 ${pi}" xyz="0.0 0.0 ${-baseshift}"/>
     </collision>
-    <xacro:default_inertial mass="10"/>
+    <xacro:default_inertial mass="4"/>
   </link>
   <joint name="base_to_basket" type="prismatic">
@@ -72,5 +84,5 @@
     </actuator>
     <joint name="base_to_basket">
-      <hardwareInterface>PositionJointInterface</hardwareInterface>
+      <hardwareInterface>hardware_interface/PositionJointInterface</hardwareInterface>
     </joint>
   </transmission>
@@ -106,4 +118,5 @@
       <kp value="10000000.0" />
       <kd value="1.0" />
+      <min_depth value="0.02" />
       <material>Gazebo/Grey</material>
     </gazebo>
@@ -116,5 +129,5 @@
       </actuator>
       <joint name="${prefix}_wheel_joint">
-        <hardwareInterface>VelocityJointInterface</hardwareInterface>
+        <hardwareInterface>hardware_interface/VelocityJointInterface</hardwareInterface>
       </joint>
     </transmission>
@@ -163,5 +176,5 @@
       </actuator>
       <joint name="${prefix}_front_wheel_joint">
-        <hardwareInterface>VelocityJointInterface</hardwareInterface>
+        <hardwareInterface>hardware_interface/VelocityJointInterface</hardwareInterface>
       </joint>
     </transmission>
@@ -169,4 +182,26 @@
    <xacro:wheel_front prefix="right" reflect="-1"/>
   <xacro:wheel_front prefix="left" reflect="1"/>
+<!-- Lidar design -->
+<joint name="scan_joint" type="fixed">
+    <parent link="base_link"/>
+    <child link="base_scan"/>
+    <origin xyz="0  ${ywheel2-0.04} ${zwheel2+0.17}" rpy="0 0 0"/>
+  </joint>
+  <link name="base_scan">
+    <visual>
+      <origin xyz="0 0 0.0" rpy="0 0 0"/>
+      <geometry>
+        <mesh filename="package://turtlebot3_description/meshes/sensors/lds.stl" scale="0.001 0.001 0.001"/>
+      </geometry>
+      <material name="black"/>
+    </visual>
+  </link>
+  <!-- IMU design -->
+  <joint name="imu_joint" type="fixed">
+    <parent link="base_link"/>
+    <child link="imu_link"/>
+    <origin xyz="0 0 ${zwheel2+0.17}" rpy="0 0 0"/>
+  </joint>
+  <link name="imu_link"/>
   <!-- Gazebo plugin for ROS Control -->
   <gazebo>
@@ -175,3 +210,72 @@
     </plugin>
   </gazebo>
+ <!-- Gazebo plugin for Lidar -->
+  <gazebo reference="base_scan">
+    <material>Gazebo/FlatBlack</material>
+    <sensor type="ray" name="lds_lfcd_sensor">
+      <pose>0 0 0 0 0 0</pose>
+      <visualize>$(arg laser_visual)</visualize>
+      <update_rate>5</update_rate>
+      <ray>
+        <scan>
+          <horizontal>
+            <samples>360</samples>
+            <resolution>1</resolution>
+            <min_angle>0.0</min_angle>
+            <max_angle>6.28319</max_angle>
+          </horizontal>
+        </scan>
+        <range>
+          <min>0.120</min>
+          <max>3.5</max>
+          <resolution>0.015</resolution>
+        </range>
+        <noise>
+          <type>gaussian</type>
+          <mean>0.0</mean>
+          <stddev>0.01</stddev>
+        </noise>
+      </ray>
+      <plugin name="gazebo_ros_lds_lfcd_controller" filename="libgazebo_ros_laser.so">
+        <topicName>scan</topicName>
+        <frameName>base_scan</frameName>
+      </plugin>
+    </sensor>
+  </gazebo>
+  <!-- Gazebo plugin for IMU -->
+  <gazebo reference="imu_link">
+    <sensor type="imu" name="imu">
+      <always_on>true</always_on>
+      <visualize>$(arg imu_visual)</visualize>
+    </sensor>
+    <material>Gazebo/FlatBlack</material>
+  </gazebo>
+  <gazebo>
+    <plugin name="imu_plugin" filename="libgazebo_ros_imu.so">
+      <alwaysOn>true</alwaysOn>
+      <bodyName>imu_link</bodyName>
+      <frameName>imu_link</frameName>
+      <topicName>imu</topicName>
+      <serviceName>imu_service</serviceName>
+      <gaussianNoise>0.0</gaussianNoise>
+      <updateRate>0</updateRate>
+      <imu>
+        <noise>
+          <type>gaussian</type>
+          <rate>
+            <mean>0.0</mean>
+            <stddev>2e-4</stddev>
+            <bias_mean>0.0000075</bias_mean>
+            <bias_stddev>0.0000008</bias_stddev>
+          </rate>
+          <accel>
+            <mean>0.0</mean>
+            <stddev>1.7e-2</stddev>
+            <bias_mean>0.1</bias_mean>
+            <bias_stddev>0.001</bias_stddev>
+          </accel>
+        </noise>
+      </imu>
+    </plugin>
+  </gazebo>
 </robot>

Commit message: project integration

File: models/shopping_cart/automatic_cart.urdf.xacro (robot description, xacro)
@@ -7,14 +7,14 @@
   <!-- Robot params -->
   <xacro:property name="baseshift" value="0.2" />
-  <xacro:property name="wheellen" value="0.025" />
+  <xacro:property name="wheellen" value="0.04" />
   <xacro:property name="wheelrad" value="0.08" />
-  <xacro:property name="wheellen2" value="0.02" />
-  <xacro:property name="wheelrad2" value="0.047" />
+  <xacro:property name="wheellen2" value="0.04" />
+  <xacro:property name="wheelrad2" value="0.08" />
   <xacro:property name="xwheel" value="0.25" />
   <xacro:property name="ywheel" value="0.2" />
   <xacro:property name="zwheel" value="-0.11" />
-  <xacro:property name="xwheel2" value="0.18" />
+  <xacro:property name="xwheel2" value="0.25" />
   <xacro:property name="ywheel2" value="-0.2" />
-  <xacro:property name="zwheel2" value="-0.15" />
+  <xacro:property name="zwheel2" value="-0.11" />
   <xacro:property name="pi" value="3.1415" />
   <!-- Sensor params -->
@@ -43,10 +43,10 @@
       <origin rpy="0 0 ${pi}" xyz="0.0 0.0 ${baseshift}"/>
     </visual>
-    <collision>
+    <!-- <collision>
       <geometry>
         <mesh filename="package://automatic_cart/models/shopping_cart/meshes/shopping_cart_base.dae"/>
       </geometry>
       <origin rpy="0 0 ${pi}" xyz="0.0 0.0 ${baseshift}"/>
-    </collision>
+    </collision> -->
     <xacro:default_inertial mass="10"/>
   </link>
@@ -54,5 +54,5 @@
     <parent link="base_footprint"/>
     <child link="base_link"/>
-    <origin xyz="0.0 0.0 0.0"/>
+    <origin rpy="0 0 ${pi/2}" xyz="0.0 0.0 0.0"/>
   </joint>
   <link name="basket">
@@ -186,5 +186,5 @@
     <parent link="base_link"/>
     <child link="base_scan"/>
-    <origin xyz="0  ${ywheel2-0.04} ${zwheel2+0.17}" rpy="0 0 0"/>
+    <origin xyz="0  ${-0.24} ${zwheel2+0.17}" rpy="0 0 0"/>
   </joint>
   <link name="base_scan">
@@ -228,5 +228,5 @@
         <range>
           <min>0.120</min>
-          <max>3.5</max>
+          <max>50.0</max>
           <resolution>0.015</resolution>
         </range>
@@ -245,5 +245,5 @@
   <!-- Gazebo plugin for IMU -->
   <gazebo reference="imu_link">
-    <sensor type="imu" name="imu">
+    <sensor type="imu" name="cart_imu">
       <always_on>true</always_on>
       <visualize>$(arg imu_visual)</visualize>
@@ -256,5 +256,5 @@
       <bodyName>imu_link</bodyName>
       <frameName>imu_link</frameName>
-      <topicName>imu</topicName>
+      <topicName>cart_imu</topicName>
       <serviceName>imu_service</serviceName>
       <gaussianNoise>0.0</gaussianNoise>

Commit message: ROS robot

File: models/shopping_cart/automatic_cart.urdf.xacro (robot description, xacro)
@@ -1,4 +1,5 @@
 <?xml version="1.0"?>
 <robot name="automatic_cart" xmlns:xacro="http://ros.org/wiki/xacro">
+  <node name="map_to_base_footprint" pkg="tf2_ros" type="static_transform_publisher" args="0 0 0 0 0 0 map base_footprint 100" />
   <!-- Colors -->
   <material name="black">
@@ -35,5 +36,5 @@
   </xacro:macro>
   <!-- Robot Design -->
-  <link name="base_footprint"/>
+  <link name="base_footprint"><frameName>base_footprint</frameName></link>
   <link name="base_link">
     <visual>
@@ -43,4 +44,5 @@
       <origin rpy="0 0 ${pi}" xyz="0.0 0.0 ${baseshift}"/>
     </visual>
+    <frameName>base_link</frameName>
     <!-- <collision>
       <geometry>
@@ -63,4 +65,5 @@
       <origin rpy="0 0 ${pi}" xyz="0.0 0.0 ${-baseshift}"/>
     </visual>
+    <frameName>basket</frameName>
     <collision>
       <geometry>
@@ -210,4 +213,17 @@
     </plugin>
   </gazebo>
+  <!-- World -->
+  <!--<gazebo>
+    <plugin name="p3d_base_controller" filename="libgazebo_ros_p3d.so">
+      <alwaysOn>true</alwaysOn>
+      <updateRate>50.0</updateRate>
+      <bodyName>base_link</bodyName>
+      <topicName>ground_truth/state</topicName>
+      <gaussianNoise>0.01</gaussianNoise>
+      <frameName>map</frameName>
+      <xyzOffsets>0 0 0</xyzOffsets>
+      <rpyOffsets>0 0 0</rpyOffsets>
+    </plugin>
+  </gazebo>-->
  <!-- Gazebo plugin for Lidar -->
   <gazebo reference="base_scan">
